File: traco_breakout_minimal.kicad_pcb (KiCad board)
At the start: 2 copper layers, 70.8 x 98.3 mm, 11 parts, among them J1 1935776, J2 Conn_01x03, J3 1935776

Commit message: Gerbers generated.
Parts:
- R1, R2: footprint Resistor_SMD:R_0603_1608Metric_Pad0.98x0.95mm_HandSolder -> Package_TO_SOT_THT:TO-220-2_Vertical
- moved R1 19.9 mm to (122.5, 65.8), turned to 90 degrees
- moved R2 7.40 mm to (139.5, 60.9), turned to -90 degrees
Routing:
- net Net-(PS1-+SENSE): track 25.2 -> 10.5 mm
- net Net-(PS1-TRIM): track 19.9 -> 33.9 mm
- net Net-(PS1--SENSE): track 11.7 -> 17.0 mm
