File: traco_breakout_minimal.kicad_sch (KiCad schematic)
At the start: 11 parts, among them J1 1935776, J2 Conn_01x03, J3 1935776

Commit message: Gerbers generated.
Parts:
- R1, R2: footprint Resistor_SMD:R_0603_1608Metric_Pad0.98x0.95mm_HandSolder -> Package_TO_SOT_THT:TO-220-2_Vertical
Other:
- note added: "Resistors need to be high power, that's why TO-220-2 resistors are used"
Changed lines of the file:
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@@
+    (effects (font (size 1.27 1.27)) (justify left bottom))
+  )
+  (text "Resistors need to be high power, that's why TO-220-2 resistors are used"
+    (at 167.005 69.85 0)
     (effects (font (size 1.27 1.27)) (justify left bottom))
   )
@@
   (label "shielding" (at 179.705 97.155 0) (fields_autoplaced)
     (effects (font (size 1.27 1.27)) (justify left bottom))
+  )
+  (symbol (lib_id "SamacSys_Parts:1935776") (at 88.265 86.36 180) (unit 1)
+    (in_bom yes) (on_board yes) (dnp no) (fields_autoplaced)
+    (property "Reference" "J1" (at 78.105 77.47 0)
+      (effects (font (size 1.27 1.27)))
+    )
+    (property "Value" "1935776" (at 78.105 80.01 0)
+      (effects (font (size 1.27 1.27)))
+    )
+    (property "Footprint" "SamacSys_Parts:1935776" (at 71.755 -8.56 0)
+      (effects (font (size 1.27 1.27)) (justify left top) hide)
+    )
+    (property "Datasheet" "https://datasheet.datasheetarchive.com/originals/distributors/SFDatasheet-2/sf-00057493.pdf" (at 71.755 -108.56 0)
+      (effects (font (size 1.27 1.27)) (justify left top) hide)
+    )
+    (property "Height" "13.65" (at 71.755 -308.56 0)
+      (effects (font (size 1.27 1.27)) (justify left top) hide)
+    )
+    (property "Manufacturer_Name" "Phoenix Contact" (at 71.755 -408.56 0)
+      (effects (font (size 1.27 1.27)) (justify left top) hide)
+    )
+    (property "Manufacturer_Part_Number" "1935776" (at 71.755 -508.56 0)
+      (effects (font (size 1.27 1.27)) (justify left top) hide)
+    )
+    (property "Mouser Part Number" "651-1935776" (at 71.755 -608.56 0)
+      (effects (font (size 1.27 1.27)) (justify left top) hide)
+    )
+    (property "Mouser Price/Stock" "https://www.mouser.co.uk/ProductDetail/Phoenix-Contact/1935776?qs=gjk32EaArKJ3oesOAo3TWA%3D%3D" (at 71.755 -708.56 0)
+      (effects (font (size 1.27 1.27)) (justify left top) hide)
+    )
+    (property "Arrow Part Number" "1935776" (at 71.755 -808.56 0)
+      (effects (font (size 1.27 1.27)) (justify left top) hide)
+    )
+    (property "Arrow Price/Stock" "https://www.arrow.com/en/products/1935776/phoenix-contact?region=nac" (at 71.755 -908.56 0)
+      (effects (font (size 1.27 1.27)) (justify left top) hide)
+    )
+    (pin "1")
+    (pin "2")
+    (instances
+      (project "traco_breakout_minimal"
+        (path "/03c49ecf-f784-4d12-9bd0-ecdf30efb896"
+          (reference "J1") (unit 1)
+        )
+      )
+    )
   )
   (symbol (lib_id "Device:R") (at 179.07 82.55 90) (unit 1)
@@
       (effects (font (size 1.27 1.27)))
     )
-    (property "Footprint" "Resistor_SMD:R_0603_1608Metric_Pad0.98x0.95mm_HandSolder" (at 179.07 84.328 90)
+    (property "Footprint" "Package_TO_SOT_THT:TO-220-2_Vertical" (at 179.07 84.328 90)
       (effects (font (size 1.27 1.27)) hide)
     )
@@
         (path "/03c49ecf-f784-4d12-9bd0-ecdf30efb896"
           (reference "R1") (unit 1)
-        )
-      )
-    )
-  )
-  (symbol (lib_id "SamacSys_Parts:1935776") (at 88.265 86.36 180) (unit 1)
-    (in_bom yes) (on_board yes) (dnp no) (fields_autoplaced)
-    (property "Reference" "J1" (at 78.105 77.47 0)
-      (effects (font (size 1.27 1.27)))
-    )
-    (property "Value" "1935776" (at 78.105 80.01 0)
-      (effects (font (size 1.27 1.27)))
-    )
-    (property "Footprint" "SamacSys_Parts:1935776" (at 71.755 -8.56 0)
-      (effects (font (size 1.27 1.27)) (justify left top) hide)
-    )
-    (property "Datasheet" "https://datasheet.datasheetarchive.com/originals/distributors/SFDatasheet-2/sf-00057493.pdf" (at 71.755 -108.56 0)
-      (effects (font (size 1.27 1.27)) (justify left top) hide)
-    )
-    (property "Height" "13.65" (at 71.755 -308.56 0)
-      (effects (font (size 1.27 1.27)) (justify left top) hide)
-    )
-    (property "Manufacturer_Name" "Phoenix Contact" (at 71.755 -408.56 0)
-      (effects (font (size 1.27 1.27)) (justify left top) hide)
-    )
-    (property "Manufacturer_Part_Number" "1935776" (at 71.755 -508.56 0)
-      (effects (font (size 1.27 1.27)) (justify left top) hide)
-    )
-    (property "Mouser Part Number" "651-1935776" (at 71.755 -608.56 0)
-      (effects (font (size 1.27 1.27)) (justify left top) hide)
-    )
-    (property "Mouser Price/Stock" "https://www.mouser.co.uk/ProductDetail/Phoenix-Contact/1935776?qs=gjk32EaArKJ3oesOAo3TWA%3D%3D" (at 71.755 -708.56 0)
-      (effects (font (size 1.27 1.27)) (justify left top) hide)
-    )
-    (property "Arrow Part Number" "1935776" (at 71.755 -808.56 0)
-      (effects (font (size 1.27 1.27)) (justify left top) hide)
-    )
-    (property "Arrow Price/Stock" "https://www.arrow.com/en/products/1935776/phoenix-contact?region=nac" (at 71.755 -908.56 0)
-      (effects (font (size 1.27 1.27)) (justify left top) hide)
-    )
-    (pin "1")
-    (pin "2")
-    (instances
-      (project "traco_breakout_minimal"
-        (path "/03c49ecf-f784-4d12-9bd0-ecdf30efb896"
-          (reference "J1") (unit 1)
         )
       )
@@
       (effects (font (size 1.27 1.27)))
     )
-    (property "Footprint" "Resistor_SMD:R_0603_1608Metric_Pad0.98x0.95mm_HandSolder" (at 179.07 89.408 90)
-      (effects (font (size 1.27 1.27)) hide)
-    )
+    (property "Footprint" "Package_TO_SOT_THT:TO-220-2_Vertical" (at 179.07 89.408 90)
+      (effects (font (size 1.27 1.27)) hide)
+    )
